File: coilgun.kicad_pcb (KiCad board)
At the start: 2 copper layers, 91.3 x 76.1 mm, 57 parts, among them J1 Conn_01x02, J2 Conn_02x05_Odd_Even, J3 Conn_02x05_Odd_Even, J4 Conn_01x03, J5 Conn_01x03, J6 Conn_01x02, J7 Conn_01x02, J8 Conn_01x02, Q1 BC547, Q2 BC557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

Commit message: text update
Parts:
- moved C10 0.59 mm to (125.2, 93.5)
Routing:
- net VDD: track 237.6 -> 236.8 mm
Other:
- board text added: "AC POWER"
- board text removed: "POWER"
Changed lines of the file:
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@@
 	(footprint "Capacitor_THT:CP_Radial_D10.0mm_P5.00mm_P7.50mm"
 		(layer "F.Cu")
-		(at 124.8 93.882677 90)
+		(at 125.25 93.5 90)
 		(descr "CP, Radial series, Radial, pin pitch=5.00mm 7.50mm, diameter=10mm, height=16mm, Electrolytic Capacitor")
 		(tags "CP Radial series Radial pin pitch 5.00mm 7.50mm diameter 10mm height 16mm Electrolytic Capacitor")
@@
 			(at 0 -3.15 0)
 			(layer "F.SilkS")
+			(hide yes)
 			(effects
 				(font
@@
 			(at 0 -3.15 0)
 			(layer "F.SilkS")
+			(hide yes)
 			(effects
 				(font
@@
 			(at 0 -3.15 0)
 			(layer "F.SilkS")
+			(hide yes)
 			(effects
 				(font
@@
 			(at 0 -3.15 0)
 			(layer "F.SilkS")
+			(hide yes)
 			(effects
 				(font
@@
 		(layer "Edge.Cuts")
 	)
-	(gr_text "Key = S1 & S2 & Safe & TRG & <maxTime"
-		(at 114.5 80.028221 0)
+	(gr_text "5V"
+		(at 143.5 97 0)
 		(layer "F.SilkS")
 		(effects
@@
 		)
 	)
-	(gr_text "15V"
-		(at 117.5 96.712677 0)
+	(gr_text "Key = S1 & S2 & Safe \n    & TRG & <maxTime"
+		(at 115 82.5 0)
 		(layer "F.SilkS")
 		(effects
 			(font
-				(size 1 1)
-				(thickness 0.1)
+				(size 1.5 1.5)
 			)
 			(justify left bottom)
 		)
 	)
-	(gr_text "5V"
-		(at 143.5 97 0)
+	(gr_text "15V"
+		(at 117.25 97.5 0)
 		(layer "F.SilkS")
 		(effects
 			(font
-				(size 1 1)
-				(thickness 0.1)
+				(size 1.5 1.5)
 			)
 			(justify left bottom)
@@
 		)
 	)
-	(gr_text "POWER"
-		(at 80.75 90.9 90)
+	(gr_text "AC POWER"
+		(at 80.75 94 90)
 		(layer "F.SilkS")
 		(effects
@@
 		(knockout no)
 	)
+	(gr_text_box "${PROJECTNAME} ${CURRENT_DATE}"
+		(start 135.666462 54.5)
+		(end 158.065625 63.819888)
+		(margins 1.0025 1.0025 1.0025 1.0025)
+		(layer "B.SilkS")
+		(effects
+			(font
+				(size 2 2)
+				(thickness 0.5)
+				(bold yes)
+			)
+			(justify left mirror)
+		)
+		(border yes)
+		(stroke
+			(width 0.1)
+			(type solid)
+		)
+		(knockout no)
+	)
 	(segment
-		(start 122.8 94.554821)
-		(end 122.8 91.782677)
-		(width 1)
+		(start 123.632677 94.554821)
+		(end 124.127856 94.554821)
+		(width 0.5)
 		(layer "F.Cu")
 		(net "VDD")
 	)
 	(segment
-		(start 131.9 97.182677)
-		(end 139.8 97.182677)
+		(start 123.25 94.172144)
+		(end 123.632677 94.554821)
+		(width 0.5)
+		(layer "F.Cu")
+		(net "VDD")
+	)
+	(segment
+		(start 125.632677 93.882677)
+		(end 128.6 93.882677)
 		(width 0.5)
 		(layer "F.Cu")
@@
 	)
 	(segment
-		(start 128.6 93.882677)
-		(end 131.9 97.182677)
-		(width 0.5)
-		(layer "F.Cu")
-		(net "VDD")
-	)
-	(segment
 		(start 117.1 73.1)
 		(end 115.42 73.1)
@@
 	)
 	(segment
-		(start 122.8 91.782677)
-		(end 119.758661 88.741339)
-		(width 1)
-		(layer "F.Cu")
-		(net "VDD")
-	)
-	(segment
 		(start 122.9 67.88)
 		(end 118.5 67.88)
@@
 	)
 	(segment
+		(start 122.8 91.782677)
+		(end 119.758661 88.741339)
+		(width 1)
+		(layer "F.Cu")
+		(net "VDD")
+	)
+	(segment
 		(start 129.5 61.6)
 		(end 129.4 61.5)
@@
 	)
 	(segment
-		(start 139.8 97.182677)
-		(end 140.6 96.382677)
-		(width 0.5)
-		(layer "F.Cu")
-		(net "VDD")
-	)
-	(segment
 		(start 115.42 73.1)
 		(end 115.28 72.96)
@@
 	)
 	(segment
-		(start 72.16 42.42)
-		(end 74.7 42.42)
-		(width 1)
+		(start 140.6 96.382677)
+		(end 140.6 94.982677)
+		(width 0.5)
 		(layer "F.Cu")
 		(net "VDD")
 	)
 	(segment
-		(start 140.6 96.382677)
-		(end 140.6 94.982677)
-		(width 0.5)
+		(start 72.16 42.42)
+		(end 74.7 42.42)
+		(width 1)
 		(layer "F.Cu")
 		(net "VDD")
@@
 	)
 	(segment
+		(start 139.8 97.182677)
+		(end 140.6 96.382677)
+		(width 0.5)
+		(layer "F.Cu")
+		(net "VDD")
+	)
+	(segment
+		(start 122.8 93.722144)
+		(end 122.8 91.782677)
+		(width 1)
+		(layer "F.Cu")
+		(net "VDD")
+	)
+	(segment
+		(start 125.25 93.5)
+		(end 125.632677 93.882677)
+		(width 0.5)
+		(layer "F.Cu")
+		(net "VDD")
+	)
+	(segment
 		(start 122.9 64.5)
 		(end 122.9 67.88)
@@
 	)
 	(segment
+		(start 128.6 93.882677)
+		(end 131.9 97.182677)
+		(width 0.5)
+		(layer "F.Cu")
+		(net "VDD")
+	)
+	(segment
 		(start 118.5 67.88)
 		(end 115.28 67.88)
@@
 	)
 	(segment
+		(start 131.9 97.182677)
+		(end 139.8 97.182677)
+		(width 0.5)
+		(layer "F.Cu")
+		(net "VDD")
+	)
+	(segment
 		(start 74.7 42.42)
 		(end 74.7 39.88)
@@
 	)
 	(segment
-		(start 122.8 94.554821)
-		(end 124.127856 94.554821)
-		(width 0.5)
+		(start 123.25 94.172144)
+		(end 122.8 93.722144)
+		(width 1)
 		(layer "F.Cu")
 		(net "VDD")
@@
 		(width 0.5)
 		(layer "F.Cu")
-		(net "VDD")
-	)
-	(segment
-		(start 124.8 93.882677)
-		(end 128.6 93.882677)
-		(width 0.5)
-		(layer "F.Cu")
